File: avr_frs_kicad/avr_frs.sch (KiCad schematic (older format))
At the start: 38 parts, among them CON1 BARREL_JACK, IC1 ATMEGA328P-P, P1 Power, P2 Analog, P3 Digital, P4 Digital, P5 CONN_1, P6 CONN_1, P7 CONN_1, P8 CONN_1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

Commit message: KiCAD circuit & PCB.
Parts:
- removed P5, P6, P7, P8: CONN_1, Socket_Arduino_Uno:Arduino_1pin, symbol CONN_1
- D1: value LED -> Red
- D3: value LED -> Green
- Q1: value Q_NPN_EBC -> 2N2222
- SW1: value SW_PUSH -> Start
Connections:
- no-connect marks 16 -> 12
Other:
- note removed: "Holes"
Changed lines of the file:
@@
 Text Label 4625 2450 0    60   ~ 0
 SCL
-$Comp
-L CONN_1 P5
-U 1 1 551BBC06
-P 4950 1975
-F 0 "P5" H 5030 1975 40  0000 L CNN
-F 1 "CONN_1" H 4950 2030 30  0001 C CNN
-F 2 "Socket_Arduino_Uno:Arduino_1pin" H 4950 1975 60  0001 C CNN
-F 3 "" H 4950 1975 60  0000 C CNN
-	1    4950 1975
-	0    -1   -1   0
-$EndComp
-$Comp
-L CONN_1 P6
-U 1 1 551BBD10
-P 5025 1975
-F 0 "P6" H 5105 1975 40  0000 L CNN
-F 1 "CONN_1" H 5025 2030 30  0001 C CNN
-F 2 "Socket_Arduino_Uno:Arduino_1pin" H 5025 1975 60  0001 C CNN
-F 3 "" H 5025 1975 60  0000 C CNN
-	1    5025 1975
-	0    -1   -1   0
-$EndComp
-$Comp
-L CONN_1 P7
-U 1 1 551BBD30
-P 5100 1975
-F 0 "P7" H 5180 1975 40  0000 L CNN
-F 1 "CONN_1" H 5100 2030 30  0001 C CNN
-F 2 "Socket_Arduino_Uno:Arduino_1pin" H 5100 1975 60  0001 C CNN
-F 3 "" H 5100 1975 60  0000 C CNN
-	1    5100 1975
-	0    -1   -1   0
-$EndComp
-$Comp
-L CONN_1 P8
-U 1 1 551BBD52
-P 5175 1975
-F 0 "P8" H 5255 1975 40  0000 L CNN
-F 1 "CONN_1" H 5175 2030 30  0001 C CNN
-F 2 "Socket_Arduino_Uno:Arduino_1pin" H 5175 1975 60  0001 C CNN
-F 3 "" H 5175 1975 60  0000 C CNN
-	1    5175 1975
-	0    -1   -1   0
-$EndComp
-Text Notes 4950 2250 0    60   ~ 0
-Holes
-NoConn ~ 4950 2125
-NoConn ~ 5025 2125
-NoConn ~ 5100 2125
-NoConn ~ 5175 2125
 Text Notes 2625 2075 0    60   ~ 0
 Shield for Arduino that uses\nthe same pin disposition\nlike "Uno" board Rev 3.
@@
 U 1 1 56E3238F
 P 4700 5400
-F 0 "Q1" H 5000 5450 50  0000 R CNN
-F 1 "Q_NPN_EBC" H 5300 5350 50  0000 R CNN
+F 0 "Q1" H 5075 5450 50  0000 R CNN
+F 1 "2N2222" H 5175 5375 50  0000 R CNN
 F 2 "TO_SOT_Packages_THT:TO-92_Horizontal2_Molded_Narrow" H 4900 5500 50  0001 C CNN
 F 3 "" H 4700 5400 50  0000 C CNN
@@
 U 1 1 56E3251F
 P 3750 5400
-F 0 "D2" H 3750 5500 50  0000 C CNN
-F 1 "12V" H 3750 5300 50  0000 C CNN
+F 0 "D2" V 3700 5250 50  0000 C CNN
+F 1 "12V" V 3800 5250 50  0000 C CNN
 F 2 "Discret:DO-35" H 3750 5400 50  0001 C CNN
 F 3 "" H 3750 5400 50  0000 C CNN
@@
 U 1 1 56E3611A
 P 4400 5100
-F 0 "R6" V 4480 5100 50  0000 C CNN
+F 0 "R6" V 4325 5100 50  0000 C CNN
 F 1 "1K" V 4400 5100 50  0000 C CNN
 F 2 "Resistors_ThroughHole:Resistor_Horizontal_RM10mm" V 4330 5100 50  0001 C CNN
@@
 U 1 1 56E372A8
 P 3500 5100
-F 0 "R5" V 3580 5100 50  0000 C CNN
+F 0 "R5" V 3425 5100 50  0000 C CNN
 F 1 "100" V 3500 5100 50  0000 C CNN
 F 2 "Resistors_ThroughHole:Resistor_Horizontal_RM7mm" V 3430 5100 50  0001 C CNN
@@
 P 2150 5200
 F 0 "D1" V 2200 5350 50  0000 C CNN
-F 1 "LED" V 2100 5350 50  0000 C CNN
+F 1 "Red" V 2100 5350 50  0000 C CNN
 F 2 "LEDs:LED-3MM" H 2150 5200 50  0001 C CNN
 F 3 "" H 2150 5200 50  0000 C CNN
@@
 U 1 1 56E373EF
 P 9350 3650
-F 0 "D3" H 9350 3750 50  0000 C CNN
-F 1 "LED" H 9350 3550 50  0000 C CNN
+F 0 "D3" V 9400 3475 50  0000 C CNN
+F 1 "Green" V 9325 3450 50  0000 C CNN
 F 2 "LEDs:LED-3MM" H 9350 3650 50  0001 C CNN
 F 3 "" H 9350 3650 50  0000 C CNN
@@
 U 1 1 56E3E6D1
 P 5550 3750
-F 0 "R9" V 5500 3600 50  0000 C CNN
+F 0 "R9" V 5500 3575 50  0000 C CNN
 F 1 "1K" V 5550 3750 50  0000 C CNN
 F 2 "Resistors_ThroughHole:Resistor_Horizontal_RM10mm" V 5480 3750 50  0001 C CNN
@@
 U 1 1 56E3E6D7
 P 5550 3850
-F 0 "R10" V 5500 3700 50  0000 C CNN
+F 0 "R10" V 5500 3675 50  0000 C CNN
 F 1 "1K" V 5550 3850 50  0000 C CNN
 F 2 "Resistors_ThroughHole:Resistor_Horizontal_RM10mm" V 5480 3850 50  0001 C CNN
@@
 U 1 1 56E3E6E9
 P 5550 4650
-F 0 "R15" V 5630 4650 50  0000 C CNN
+F 0 "R15" V 5475 4650 50  0000 C CNN
 F 1 "1K" V 5550 4650 50  0000 C CNN
 F 2 "Resistors_ThroughHole:Resistor_Horizontal_RM10mm" V 5480 4650 50  0001 C CNN
@@
 U 1 1 56E3E6EF
 P 5550 4800
-F 0 "R16" V 5630 4800 50  0000 C CNN
+F 0 "R16" V 5475 4800 50  0000 C CNN
 F 1 "1K" V 5550 4800 50  0000 C CNN
 F 2 "Resistors_ThroughHole:Resistor_Horizontal_RM10mm" V 5480 4800 50  0001 C CNN
@@
 U 1 1 56E3E7B5
 P 3400 5850
-F 0 "R4" V 3480 5850 50  0000 C CNN
+F 0 "R4" V 3325 5850 50  0000 C CNN
 F 1 "1K" V 3400 5850 50  0000 C CNN
 F 2 "Resistors_ThroughHole:Resistor_Horizontal_RM7mm" V 3330 5850 50  0001 C CNN
@@
 U 1 1 56E4D86E
 P 5550 3950
-F 0 "R11" V 5500 3800 50  0000 C CNN
+F 0 "R11" V 5500 3775 50  0000 C CNN
 F 1 "1K" V 5550 3950 50  0000 C CNN
 F 2 "Resistors_ThroughHole:Resistor_Horizontal_RM10mm" V 5480 3950 50  0001 C CNN
@@
 U 1 1 56E4D874
 P 5550 4050
-F 0 "R12" V 5500 3900 50  0000 C CNN
+F 0 "R12" V 5500 3875 50  0000 C CNN
 F 1 "1K" V 5550 4050 50  0000 C CNN
 F 2 "Resistors_ThroughHole:Resistor_Horizontal_RM10mm" V 5480 4050 50  0001 C CNN
@@
 U 1 1 56E4D8EC
 P 5550 4150
-F 0 "R13" V 5500 4000 50  0000 C CNN
+F 0 "R13" V 5500 3975 50  0000 C CNN
 F 1 "1K" V 5550 4150 50  0000 C CNN
 F 2 "Resistors_ThroughHole:Resistor_Horizontal_RM10mm" V 5480 4150 50  0001 C CNN
@@
 U 1 1 56E4D8F2
 P 5550 4250
-F 0 "R14" V 5500 4100 50  0000 C CNN
+F 0 "R14" V 5500 4075 50  0000 C CNN
 F 1 "1K" V 5550 4250 50  0000 C CNN
 F 2 "Resistors_ThroughHole:Resistor_Horizontal_RM10mm" V 5480 4250 50  0001 C CNN
@@
 U 1 1 56E4FE74
 P 5550 3550
-F 0 "R7" V 5500 3400 50  0000 C CNN
+F 0 "R7" V 5500 3375 50  0000 C CNN
 F 1 "1K" V 5550 3550 50  0000 C CNN
 F 2 "Resistors_ThroughHole:Resistor_Horizontal_RM10mm" V 5480 3550 50  0001 C CNN
@@
 U 1 1 56E4FF29
 P 5550 3650
-F 0 "R8" V 5500 3500 50  0000 C CNN
+F 0 "R8" V 5500 3475 50  0000 C CNN
 F 1 "1K" V 5550 3650 50  0000 C CNN
 F 2 "Resistors_ThroughHole:Resistor_Horizontal_RM10mm" V 5480 3650 50  0001 C CNN
@@
 U 1 1 56E4FFAD
 P 5700 3150
-F 0 "R20" V 5650 3000 50  0000 C CNN
+F 0 "R20" V 5650 2975 50  0000 C CNN
 F 1 "1K" V 5700 3150 50  0000 C CNN
 F 2 "Resistors_ThroughHole:Resistor_Horizontal_RM10mm" V 5630 3150 50  0001 C CNN
@@
 U 1 1 56E4FFB3
 P 5700 3250
-F 0 "R21" V 5650 3100 50  0000 C CNN
+F 0 "R21" V 5650 3075 50  0000 C CNN
 F 1 "1K" V 5700 3250 50  0000 C CNN
 F 2 "Resistors_ThroughHole:Resistor_Horizontal_RM10mm" V 5630 3250 50  0001 C CNN
@@
 U 1 1 56E514CF
 P 5700 2950
-F 0 "R18" V 5650 2800 50  0000 C CNN
+F 0 "R18" V 5650 2775 50  0000 C CNN
 F 1 "1K" V 5700 2950 50  0000 C CNN
 F 2 "Resistors_ThroughHole:Resistor_Horizontal_RM10mm" V 5630 2950 50  0001 C CNN
@@
 U 1 1 56E514D5
 P 5700 3050
-F 0 "R19" V 5650 2900 50  0000 C CNN
+F 0 "R19" V 5650 2875 50  0000 C CNN
 F 1 "1K" V 5700 3050 50  0000 C CNN
 F 2 "Resistors_ThroughHole:Resistor_Horizontal_RM10mm" V 5630 3050 50  0001 C CNN
@@
 U 1 1 56E515BF
 P 2400 2950
-F 0 "R3" V 2350 2800 50  0000 C CNN
+F 0 "R3" V 2325 2950 50  0000 C CNN
 F 1 "1K" V 2400 2950 50  0000 C CNN
 F 2 "Resistors_ThroughHole:Resistor_Horizontal_RM10mm" V 2330 2950 50  0001 C CNN
@@
 U 1 1 56E515C5
 P 5700 2850
-F 0 "R17" V 5650 2700 50  0000 C CNN
+F 0 "R17" V 5650 2675 50  0000 C CNN
 F 1 "1K" V 5700 2850 50  0000 C CNN
 F 2 "Resistors_ThroughHole:Resistor_Horizontal_RM10mm" V 5630 2850 50  0001 C CNN
@@
 U 1 1 56E515CB
 P 2150 4550
-F 0 "R2" V 2100 4400 50  0000 C CNN
+F 0 "R2" V 2075 4550 50  0000 C CNN
 F 1 "1K" V 2150 4550 50  0000 C CNN
 F 2 "Resistors_ThroughHole:Resistor_Horizontal_RM7mm" V 2080 4550 50  0001 C CNN
@@
 U 1 1 56E515D1
 P 2150 2950
-F 0 "R1" V 2100 2800 50  0000 C CNN
+F 0 "R1" V 2075 2950 50  0000 C CNN
 F 1 "1K" V 2150 2950 50  0000 C CNN
 F 2 "Resistors_ThroughHole:Resistor_Horizontal_RM10mm" V 2080 2950 50  0001 C CNN
@@
 	3475 3450 3400 3450
 Connection ~ 3400 3450
-Wire Notes Line
-	5300 2300 4850 2300
-Wire Notes Line
-	4850 2300 4850 1800
 Wire Notes Line
 	5300 4550 2600 4550
@@
 U 1 1 56E5E45B
 P 1900 4300
-F 0 "SW1" H 2050 4410 50  0000 C CNN
-F 1 "SW_PUSH" H 1900 4220 50  0000 C CNN
+F 0 "SW1" V 1925 4550 50  0000 C CNN
+F 1 "Start" V 1850 4550 50  0000 C CNN
 F 2 "Buttons_Switches_ThroughHole:SW_PUSH_SMALL" H 1900 4300 50  0001 C CNN
 F 3 "" H 1900 4300 50  0000 C CNN
@@
 NoConn ~ 5200 2650
 NoConn ~ 3200 5200
+Wire Notes Line
+	5300 4550 5300 1800
+Wire Notes Line
+	5300 1800 2600 1800
 $EndSCHEMATC
