File: avr_frs_kicad/avr_frs.kicad_pcb (KiCad board)
At the start: 2 copper layers, 68.6 x 53.3 mm, 38 parts, among them CON1 BARREL_JACK, IC1 ATMEGA328P-P, P1 Power, P2 Analog, P3 Digital, P4 Digital, P5 CONN_1, P6 CONN_1, P7 CONN_1, P8 CONN_1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

Commit message: KiCAD circuit & PCB.
Parts:
- removed P5, P6, P7, P8: CONN_1, Socket_Arduino_Uno:Arduino_1pin
Changed lines of the file:
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@@
     (links 62)
     (no_connects 1)
-    (area 110.922999 72.949999 179.653001 126.440001)
+    (area 104.572999 72.949999 179.653001 126.440001)
     (thickness 1.6)
     (drawings 26)
     (tracks 228)
     (zones 0)
-    (modules 38)
+    (modules 34)
     (nets 45)
   )
@@
     (visible_elements 7FFFFFFF)
     (pcbplotparams
-      (layerselection 0x00030_80000001)
+      (layerselection 0x01000_80000000)
       (usegerberextensions false)
-      (excludeedgelayer true)
+      (excludeedgelayer false)
       (linewidth 0.100000)
       (plotframeref false)
@@
       (plotvalue true)
       (plotinvisibletext false)
-      (padsonsilk false)
+      (padsonsilk true)
       (subtractmaskfromsilk false)
-      (outputformat 1)
+      (outputformat 5)
       (mirror false)
       (drillshape 1)
@@
     (add_net "Net-(Q1-Pad2)")
   )
-  (module Socket_Arduino_Uno:Arduino_1pin (layer F.Cu)
-    (at 122.428 85.725)
-    (descr "module 1 pin (ou trou mecanique de percage)")
-    (tags DEV)
-    (fp_text reference P6 (at 0 -3.048) (layer F.SilkS) hide
-      (effects (font (size 1 1) (thickness 0.15)))
-    )
-    (fp_text value CONN_1 (at 0 2.794) (layer F.Fab) hide
-      (effects (font (size 1 1) (thickness 0.15)))
-    )
-    (fp_circle (center 0 0) (end 0 -2.286) (layer F.SilkS) (width 0.15))
-    (pad 1 thru_hole circle (at 0 0) (size 4.064 4.064) (drill 3.048) (layers *.Cu *.Mask F.SilkS))
-  )
   (module Resistors_ThroughHole:Resistor_Horizontal_RM10mm placed (layer F.Cu)
     (at 177.038 99.695 90)
@@
       (effects (font (size 1 1) (thickness 0.15)))
     )
-    (fp_text value 1K (at 5.08 3.81 90) (layer F.Fab)
+    (fp_text value 1K (at 5.08 0 90) (layer F.Fab)
       (effects (font (size 1 1) (thickness 0.15)))
     )
@@
     )
   )
-  (module Socket_Arduino_Uno:Arduino_1pin (layer F.Cu)
-    (at 116.078 85.725)
-    (descr "module 1 pin (ou trou mecanique de percage)")
-    (tags DEV)
-    (fp_text reference P5 (at 0 -3.048) (layer F.SilkS) hide
-      (effects (font (size 1 1) (thickness 0.15)))
-    )
-    (fp_text value CONN_1 (at 0 2.794) (layer F.Fab) hide
-      (effects (font (size 1 1) (thickness 0.15)))
-    )
-    (fp_circle (center 0 0) (end 0 -2.286) (layer F.SilkS) (width 0.15))
-    (pad 1 thru_hole circle (at 0 0) (size 4.064 4.064) (drill 3.048) (layers *.Cu *.Mask F.SilkS))
-  )
-  (module Socket_Arduino_Uno:Arduino_1pin locked (layer F.Cu)
-    (at 126.238 75.565)
-    (descr "module 1 pin (ou trou mecanique de percage)")
-    (tags DEV)
-    (fp_text reference P7 (at 0 -3.048) (layer F.SilkS) hide
-      (effects (font (size 1 1) (thickness 0.15)))
-    )
-    (fp_text value CONN_1 (at 0 2.794) (layer F.Fab) hide
-      (effects (font (size 1 1) (thickness 0.15)))
-    )
-    (fp_circle (center 0 0) (end 0 -2.286) (layer F.SilkS) (width 0.15))
-    (pad 1 thru_hole circle (at 0 0) (size 4.064 4.064) (drill 3.048) (layers *.Cu *.Mask F.SilkS))
-  )
-  (module Socket_Arduino_Uno:Arduino_1pin (layer F.Cu)
-    (at 116.078 75.565)
-    (descr "module 1 pin (ou trou mecanique de percage)")
-    (tags DEV)
-    (fp_text reference P8 (at 0 -3.048) (layer F.SilkS) hide
-      (effects (font (size 1 1) (thickness 0.15)))
-    )
-    (fp_text value CONN_1 (at 0 2.794) (layer F.Fab) hide
-      (effects (font (size 1 1) (thickness 0.15)))
-    )
-    (fp_circle (center 0 0) (end 0 -2.286) (layer F.SilkS) (width 0.15))
-    (pad 1 thru_hole circle (at 0 0) (size 4.064 4.064) (drill 3.048) (layers *.Cu *.Mask F.SilkS))
-  )
   (module Capacitors_ThroughHole:C_Radial_D5_L6_P2.5 placed (layer F.Cu)

Commit message: Minor rerouting.
Parts:
- moved R1 1.80 mm to (149.1, 107.3)
Routing:
- net Net-(IC1-Pad6): track 45.1 -> 41.5 mm
- net /A2: track 20.1 -> 22.6 mm
- net Net-(IC1-Pad5): track 37.1 -> 34.9 mm
- net GNDREF: track 178.1 -> 175.9 mm
- net Net-(IC1-Pad25): track 16.3 -> 14.8 mm
Changed lines of the file:
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@@
-(kicad_pcb (version 4) (host pcbnew 4.0.1-stable)
+(kicad_pcb (version 4) (host pcbnew 4.0.2-stable)
   (general
     (links 62)
     (no_connects 1)
-    (area 104.572999 72.949999 179.653001 126.440001)
+    (area 110.922999 72.949999 179.653001 126.440001)
     (thickness 1.6)
     (drawings 26)
-    (tracks 228)
+    (tracks 221)
     (zones 0)
     (modules 34)
@@
   )
   (setup
-    (last_trace_width 0.25)
+    (last_trace_width 0.75)
     (user_trace_width 0.5)
     (user_trace_width 0.75)
@@
   )
   (module Resistors_ThroughHole:Resistor_Horizontal_RM10mm placed (layer F.Cu)
-    (at 150.368 108.585)
+    (at 149.098 107.315)
     (descr "Resistor, Axial,  RM 10mm, 1/3W")
     (tags "Resistor Axial RM 10mm 1/3W")
@@
   (segment (start 164.338 112.395) (end 164.338 120.015) (width 0.75) (layer B.Cu) (net 2))
   (segment (start 164.338 120.015) (end 164.338 123.825) (width 0.75) (layer B.Cu) (net 2))
-  (segment (start 166.878 123.825) (end 166.878 111.125) (width 0.75) (layer B.Cu) (net 3))
-  (segment (start 164.338 108.585) (end 160.528 108.585) (width 0.75) (layer B.Cu) (net 3))
-  (segment (start 166.878 111.125) (end 164.338 108.585) (width 0.75) (layer B.Cu) (net 3))
+  (segment (start 166.878 123.825) (end 166.878 109.855) (width 0.75) (layer B.Cu) (net 3))
+  (segment (start 164.338 107.315) (end 159.258 107.315) (width 0.75) (layer B.Cu) (net 3))
+  (segment (start 166.878 109.855) (end 164.338 107.315) (width 0.75) (layer B.Cu) (net 3))
   (segment (start 169.418 118.745) (end 169.418 123.825) (width 0.75) (layer B.Cu) (net 4))
   (segment (start 171.958 118.745) (end 171.958 123.825) (width 0.75) (layer B.Cu) (net 5))
@@
   (segment (start 116.078 99.695) (end 117.348 100.965) (width 0.75) (layer B.Cu) (net 21))
   (segment (start 116.078 93.345) (end 116.078 97.155) (width 0.75) (layer B.Cu) (net 21))
+  (segment (start 159.258 112.395) (end 156.718 109.855) (width 0.75) (layer B.Cu) (net 22))
+  (segment (start 156.718 104.775) (end 156.718 102.235) (width 0.75) (layer B.Cu) (net 22))
+  (segment (start 156.718 104.775) (end 156.718 109.855) (width 0.75) (layer B.Cu) (net 22))
+  (segment (start 114.808 80.645) (end 112.268 83.185) (width 1.5) (layer B.Cu) (net 22))
+  (segment (start 127.508 80.645) (end 114.808 80.645) (width 1.5) (layer B.Cu) (net 22))
+  (segment (start 130.048 78.105) (end 127.508 80.645) (width 1.5) (layer B.Cu) (net 22))
+  (segment (start 136.398 78.105) (end 130.048 78.105) (width 1.5) (layer B.Cu) (net 22))
+  (segment (start 137.414 77.089) (end 136.398 78.105) (width 1.5) (layer B.Cu) (net 22))
+  (segment (start 137.414 75.565) (end 137.414 77.089) (width 1.5) (layer B.Cu) (net 22))
+  (segment (start 112.268 83.185) (end 112.268 90.845) (width 1.5) (layer B.Cu) (net 22))
   (segment (start 115.64366 111.76) (end 112.268 111.76) (width 1.5) (layer B.Cu) (net 22))
   (segment (start 116.078 90.845) (end 118.578 90.845) (width 0.75) (layer B.Cu) (net 22))
@@
   (segment (start 112.268 109.855) (end 112.268 104.775) (width 1.5) (layer B.Cu) (net 22))
   (segment (start 112.268 104.775) (end 112.268 90.845) (width 1.5) (layer B.Cu) (net 22))
-  (segment (start 112.268 90.845) (end 112.268 83.185) (width 1.5) (layer B.Cu) (net 22))
   (segment (start 114.808 120.015) (end 112.268 117.475) (width 1.5) (layer B.Cu) (net 22))
   (segment (start 132.588 116.205) (end 132.588 120.015) (width 0.75) (layer B.Cu) (net 22))
-  (segment (start 137.414 75.565) (end 137.414 77.089) (width 1.5) (layer B.Cu) (net 22))
-  (segment (start 137.414 77.089) (end 136.398 78.105) (width 1.5) (layer B.Cu) (net 22))
-  (segment (start 136.398 78.105) (end 130.048 78.105) (width 1.5) (layer B.Cu) (net 22))
-  (segment (start 130.048 78.105) (end 127.508 80.645) (width 1.5) (layer B.Cu) (net 22))
-  (segment (start 127.508 80.645) (end 112.268 80.645) (width 1.5) (layer B.Cu) (net 22))
-  (segment (start 112.268 80.645) (end 112.268 83.185) (width 1.5) (layer B.Cu) (net 22))
   (segment (start 137.668 120.015) (end 132.588 120.015) (width 1.5) (layer B.Cu) (net 22))
   (segment (start 137.668 117.475) (end 137.668 120.015) (width 0.75) (layer B.Cu) (net 22))
@@
   (segment (start 149.098 97.155) (end 152.908 97.155) (width 0.75) (layer B.Cu) (net 22))
   (segment (start 152.908 97.155) (end 154.178 97.155) (width 0.75) (layer B.Cu) (net 22))
-  (segment (start 156.718 102.235) (end 156.718 111.125) (width 1) (layer B.Cu) (net 22))
-  (segment (start 157.988 112.395) (end 159.258 112.395) (width 1) (layer B.Cu) (net 22))
-  (segment (start 156.718 111.125) (end 157.988 112.395) (width 1) (layer B.Cu) (net 22))
   (segment (start 151.638 123.825) (end 154.178 123.825) (width 0.75) (layer B.Cu) (net 22))
   (segment (start 116.078 104.775) (end 116.078 106.045) (width 0.75) (layer B.Cu) (net 23))
@@
   (segment (start 132.588 98.425) (end 133.858 99.695) (width 0.75) (layer B.Cu) (net 28))
   (segment (start 132.588 94.615) (end 132.588 98.425) (width 0.75) (layer B.Cu) (net 28))
+  (segment (start 127.508 100.965) (end 128.778 102.235) (width 0.75) (layer B.Cu) (net 29))
+  (segment (start 128.778 102.235) (end 128.778 107.315) (width 0.75) (layer B.Cu) (net 29))
+  (segment (start 128.778 107.315) (end 130.048 108.585) (width 0.75) (layer B.Cu) (net 29))
+  (segment (start 130.048 108.585) (end 144.018 108.585) (width 0.75) (layer B.Cu) (net 29))
   (segment (start 127.508 97.155) (end 127.508 100.965) (width 0.75) (layer B.Cu) (net 29))
-  (segment (start 149.098 106.045) (end 149.098 102.235) (width 0.75) (layer B.Cu) (net 29))
-  (segment (start 147.828 107.315) (end 149.098 106.045) (width 0.75) (layer B.Cu) (net 29))
-  (segment (start 147.828 108.585) (end 147.828 107.315) (width 0.75) (layer B.Cu) (net 29))
-  (segment (start 130.048 108.585) (end 147.828 108.585) (width 0.75) (layer B.Cu) (net 29))
-  (segment (start 128.778 107.315) (end 130.048 108.585) (width 0.75) (layer B.Cu) (net 29))
-  (segment (start 128.778 102.235) (end 128.778 107.315) (width 0.75) (layer B.Cu) (net 29))
-  (segment (start 127.508 100.965) (end 128.778 102.235) (width 0.75) (layer B.Cu) (net 29))
+  (segment (start 149.098 103.505) (end 149.098 102.235) (width 0.75) (layer B.Cu) (net 29))
+  (segment (start 144.018 108.585) (end 149.098 103.505) (width 0.75) (layer B.Cu) (net 29))
   (segment (start 123.698 100.965) (end 126.238 103.505) (width 0.75) (layer B.Cu) (net 30))
-  (segment (start 151.638 106.045) (end 151.638 102.235) (width 0.75) (layer B.Cu) (net 30))
-  (segment (start 152.908 107.315) (end 151.638 106.045) (width 0.75) (layer B.Cu) (net 30))
-  (segment (start 152.908 108.585) (end 152.908 107.315) (width 0.75) (layer B.Cu) (net 30))
-  (segment (start 152.908 109.855) (end 152.908 108.585) (width 0.75) (layer B.Cu) (net 30))
-  (segment (start 151.638 111.125) (end 152.908 109.855) (width 0.75) (layer B.Cu) (net 30))
-  (segment (start 150.368 111.125) (end 151.638 111.125) (width 0.75) (layer B.Cu) (net 30))
-  (segment (start 149.098 111.125) (end 150.368 111.125) (width 0.75) (layer B.Cu) (net 30))
-  (segment (start 147.828 109.855) (end 149.098 111.125) (width 0.75) (layer B.Cu) (net 30))
+  (segment (start 151.638 108.585) (end 151.638 102.235) (width 0.75) (layer B.Cu) (net 30))
+  (segment (start 150.368 109.855) (end 151.638 108.585) (width 0.75) (layer B.Cu) (net 30))
+  (segment (start 149.098 109.855) (end 150.368 109.855) (width 0.75) (layer B.Cu) (net 30))
+  (segment (start 147.828 109.855) (end 149.098 109.855) (width 0.75) (layer B.Cu) (net 30))
   (segment (start 127.508 109.855) (end 147.828 109.855) (width 0.75) (layer B.Cu) (net 30))
   (segment (start 126.238 108.585) (end 127.508 109.855) (width 0.75) (layer B.Cu) (net 30))
@@
   (segment (start 151.638 90.805) (end 152.908 89.535) (width 0.75) (layer B.Cu) (net 42))
   (segment (start 149.098 93.345) (end 151.638 90.805) (width 0.75) (layer B.Cu) (net 42))
-  (segment (start 150.368 108.585) (end 150.368 103.505) (width 0.75) (layer B.Cu) (net 43))
+  (segment (start 150.368 103.505) (end 150.368 100.965) (width 0.5) (layer B.Cu) (net 43))
+  (segment (start 150.368 100.965) (end 146.558 97.155) (width 0.75) (layer B.Cu) (net 43))
   (segment (start 146.558 97.155) (end 146.558 94.615) (width 0.75) (layer B.Cu) (net 43))
-  (segment (start 147.828 98.425) (end 146.558 97.155) (width 0.75) (layer B.Cu) (net 43))
-  (segment (start 149.098 98.425) (end 147.828 98.425) (width 0.75) (layer B.Cu) (net 43))
-  (segment (start 150.368 99.695) (end 149.098 98.425) (width 0.75) (layer B.Cu) (net 43))
-  (segment (start 150.368 100.965) (end 150.368 99.695) (width 0.75) (layer B.Cu) (net 43))
-  (segment (start 150.368 103.505) (end 150.368 100.965) (width 0.5) (layer B.Cu) (net 43))
+  (segment (start 150.368 106.045) (end 150.368 103.505) (width 0.75) (layer B.Cu) (net 43))
+  (segment (start 149.098 107.315) (end 150.368 106.045) (width 0.75) (layer B.Cu) (net 43))
   (segment (start 144.018 114.935) (end 133.858 114.935) (width 0.75) (layer B.Cu) (net 44))
 )
